File: HARDWARE/KICAD/PCB/piano_electronico/piano_electronico.kicad_sch (KiCad schematic)
At the start: 1 part, among them U1 LM555xM

Commit message: rev3
Parts:
- added U2: ~, symbol hueso:HUESO
Changed lines of the file:
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@@
+		)
+	)
+	(symbol
+		(lib_id "hueso:HUESO")
+		(at 127 48.26 0)
+		(unit 1)
+		(exclude_from_sim no)
+		(in_bom yes)
+		(on_board yes)
+		(dnp no)
+		(fields_autoplaced yes)
+		(property "Reference" "U2"
+			(at 127.635 39.37 0)
+			(effects
+				(font
+					(size 1.27 1.27)
+				)
+			)
+		)
+		(property "Value" "~"
+			(at 127.635 41.91 0)
+			(effects
+				(font
+					(size 1.27 1.27)
+				)
+			)
+		)
+		(property "Footprint" ""
+			(at 127 48.26 0)
+			(effects
+				(font
+					(size 1.27 1.27)
+				)
+				(hide yes)
+			)
+		)
+		(property "Datasheet" ""
+			(at 127 48.26 0)
+			(effects
+				(font
+					(size 1.27 1.27)
+				)
+				(hide yes)
+			)
+		)
+		(property "Description" ""
+			(at 127 48.26 0)
+			(effects
+				(font
+					(size 1.27 1.27)
+				)
+				(hide yes)
+			)
+		)
+		(pin ""
+		)
+		(pin ""
+		)
+		(instances
+			(project ""
+				(path "/478d9700-87ed-4f57-bca2-65adb743de24"
+					(reference "U2")
+					(unit 1)
+				)
+			)
 		)
 	)
